Commit message: inverse kinematics + transformation matrix

File: sophia_description/urdf/mech/leg.urdf.xacro (robot description, xacro)
@@ -112,5 +112,5 @@
     <joint name="${prefix}coxa_link_to_${prefix}femur_link" type="revolute">
       <axis xyz="0 1 0"/>
-      <limit effort="${joint_effort}" lower="-1.57" upper="1.57" velocity="${joint_velocity}"/>
+      <limit effort="${joint_effort}" lower="-2.5" upper="2.5" velocity="${joint_velocity}"/>
       <parent link="${prefix}coxa_link"/>
       <child link="${prefix}femur_link"/>
@@ -120,5 +120,5 @@
     <joint name="${prefix}femur_link_to_${prefix}tibia_link" type="revolute">
       <axis xyz="0 1 0"/>
-      <limit effort="${joint_effort}" lower="-1.57" upper="1.57" velocity="${joint_velocity}"/>
+      <limit effort="${joint_effort}" lower="-2.0" upper="2.0" velocity="${joint_velocity}"/>
       <parent link="${prefix}femur_link"/>
       <child link="${prefix}tibia_link"/>
@@ -126,4 +126,11 @@
       <dynamics damping="${joint_damping}" friction="${joint_friction}"/>
     </joint>
+    <gazebo reference="${prefix}tibia_link">
+      <mu1 value="2.0"/>
+      <mu2 value="2.0"/>
+      <kp value="10000000.0"/>
+      <kd value="1.0"/>
+      <minDepth value="0.001"/>
+    </gazebo>
     <xacro:material_visual ref_link="${prefix}coxa_link" ambient="1 1 1 1" diffuse="1 1 1 1" specular="1 1 1 1"/>
     <xacro:material_visual ref_link="${prefix}femur_link" ambient="1 1 1 1" diffuse="1 1 1 1" specular="1 1 1 1"/>

Commit message: walk task with bezier cubic curve

File: sophia_description/urdf/mech/leg.urdf.xacro (robot description, xacro)
@@ -1,5 +1,5 @@
 <?xml version="1.0"?>
 <robot xmlns:xacro="http://www.ros.org/wiki/xacro">
-    <xacro:property name="joint_effort" value="3.0"/>  <!-- max torque -->
+    <xacro:property name="joint_effort" value="15.0"/>  <!-- max torque -->
     <xacro:property name="joint_velocity" value="2.792527"/>
     <xacro:property name="joint_damping" value="0.1"/>
@@ -127,9 +127,9 @@
     </joint>
     <gazebo reference="${prefix}tibia_link">
-      <mu1 value="2.0"/>
-      <mu2 value="2.0"/>
-      <kp value="10000000.0"/>
-      <kd value="1.0"/>
-      <minDepth value="0.001"/>
+      <mu1>2.0</mu1>
+      <mu2>2.0</mu2>
+      <kp>1000000.0</kp>
+      <kd>100.0</kd>
+      <minDepth>0.001</minDepth>
     </gazebo>
     <xacro:material_visual ref_link="${prefix}coxa_link" ambient="1 1 1 1" diffuse="1 1 1 1" specular="1 1 1 1"/>

Commit message: read xacro config + launch joystick nodes automation

File: sophia_description/urdf/mech/leg.urdf.xacro (robot description, xacro)
@@ -6,15 +6,16 @@
     <xacro:property name="joint_friction" value="0.01"/>
     <xacro:property name="coxa_link_mass" value="0.05"/>
-    <xacro:property name="coxa_link_width" value="0.04"/>
-    <xacro:property name="coxa_link_height" value="0.04"/>
-    <xacro:property name="coxa_link_depth" value="0.04"/>
+    <xacro:property name="coxa_link_width" value="0.035"/>
+    <xacro:property name="coxa_link_height" value="0.045"/>
+    <xacro:property name="coxa_link_depth" value="0.042"/>
     <xacro:property name="femur_link_mass" value="0.10"/>
-    <xacro:property name="femur_link_width" value="0.10"/>
-    <xacro:property name="femur_link_height" value="0.03"/>
-    <xacro:property name="femur_link_depth" value="0.03"/>
+    <xacro:property name="femur_link_width" value="0.045"/>
+    <xacro:property name="femur_link_height" value="0.013"/>
+    <xacro:property name="femur_link_depth" value="0.025"/>
     <xacro:property name="tibia_link_mass" value="0.08"/>
-    <xacro:property name="tibia_link_width" value="0.15"/>
-    <xacro:property name="tibia_link_height" value="0.02"/>
-    <xacro:property name="tibia_link_depth" value="0.02"/>
+    <xacro:property name="tibia_link_width" value="0.09"/>
+    <xacro:property name="tibia_link_height" value="0.015"/>
+    <xacro:property name="tibia_link_depth" value="0.005"/>
+    <xacro:property name="tibia_sphere_radius" value="${tibia_link_height/2}"/>
     <xacro:macro name="link_inertial" params="m w h d">
         <inertial>
@@ -42,14 +43,11 @@
       <visual>
         <geometry>
-          <box size="${coxa_link_width} ${coxa_link_height} ${coxa_link_depth}"/>
+          <box size="${coxa_link_width} ${coxa_link_depth} ${coxa_link_height}"/>
         </geometry>
         <origin xyz="${coxa_link_width/2} 0.0 0.0" rpy="0 0 0"/>
-        <material name="white">
-          <color rgba="1 1 1 1"/>
-        </material>
       </visual>
       <collision>
         <geometry>
-          <box size="${coxa_link_width} ${coxa_link_height} ${coxa_link_depth}"/>
+          <box size="${coxa_link_width} ${coxa_link_depth} ${coxa_link_height}"/>
         </geometry>
         <origin xyz="${coxa_link_width/2} 0.0 0.0" rpy="0 0 0"/>
@@ -60,14 +58,11 @@
       <visual>
         <geometry>
-          <box size="${femur_link_width} ${femur_link_height} ${femur_link_depth}"/>
+          <box size="${femur_link_width} ${femur_link_depth} ${femur_link_height}"/>
         </geometry>
         <origin xyz="${femur_link_width/2} 0.0 0.0" rpy="0 0 0"/>
-        <material name="white">
-          <color rgba="1 1 1 1"/>
-        </material>
       </visual>
       <collision>
         <geometry>
-          <box size="${femur_link_width} ${femur_link_height} ${femur_link_depth}"/>
+          <box size="${femur_link_width} ${femur_link_depth} ${femur_link_height}"/>
         </geometry>
         <origin xyz="${femur_link_width/2} 0.0 0.0" rpy="0 0 0"/>
@@ -78,16 +73,19 @@
       <visual>
         <geometry>
-          <box size="${tibia_link_width} ${tibia_link_height} ${tibia_link_depth}"/>
+          <box size="${tibia_link_width} ${tibia_link_depth} ${tibia_link_height}"/>
         </geometry>
         <origin xyz="${tibia_link_width/2} 0.0 0.0" rpy="0 0 0"/>
-        <material name="white">
-          <color rgba="1 1 1 1"/>
-        </material>
       </visual>
-      <collision>
+      <collision name="${prefix}tibia_body_collision">
         <geometry>
-          <box size="${tibia_link_width} ${tibia_link_height} ${tibia_link_depth}"/>
+          <box size="${tibia_link_width - tibia_sphere_radius} ${tibia_link_depth} ${tibia_link_height}"/>
         </geometry>
-        <origin xyz="${tibia_link_width/2} 0.0 0.0" rpy="0 0 0"/>
+        <origin xyz="${(tibia_link_width - tibia_sphere_radius)/2} 0.0 0.0" rpy="0 0 0"/>
+      </collision>
+      <collision name="${prefix}tibia_foot_collision">
+        <geometry>
+          <sphere radius="${tibia_sphere_radius}"/>
+        </geometry>
+        <origin xyz="${tibia_link_width - tibia_sphere_radius} 0.0 0.0" rpy="0 0 0"/>
       </collision>
     </link>
@@ -127,9 +125,9 @@
     </joint>
     <gazebo reference="${prefix}tibia_link">
-      <mu1>2.0</mu1>
-      <mu2>2.0</mu2>
-      <kp>1000000.0</kp>
-      <kd>100.0</kd>
-      <minDepth>0.001</minDepth>
+      <mu1>1.5</mu1>
+      <mu2>1.5</mu2>
+      <kp>500000.0</kp>
+      <kd>10.0</kd>
+      <minDepth>0.002</minDepth>
     </gazebo>
     <xacro:material_visual ref_link="${prefix}coxa_link" ambient="1 1 1 1" diffuse="1 1 1 1" specular="1 1 1 1"/>

File: sophia_description/urdf/mech/prosoma_chassis.urdf.xacro (robot description, xacro)
@@ -2,7 +2,6 @@
 <robot xmlns:xacro="http://wiki.ros.org/xacro">
     <xacro:property name="chassis_mass" value="0.5"/>
-    <xacro:property name="chassis_width" value="0.12"/>
-    <xacro:property name="chassis_length" value="0.20"/>
-    <xacro:property name="chassis_height" value="0.03"/>
+    <xacro:property name="chassis_radius" value="0.06"/>
+    <xacro:property name="chassis_height" value="0.045"/>
     <xacro:macro name="prosoma_chassis" params="base_link prefix">
         <link name="${prefix}${base_link}">
@@ -11,11 +10,11 @@
                 <mass value="${chassis_mass}"/>
                 <inertia
-                    ixx="${(1/12) * chassis_mass * (chassis_length**2 + chassis_height**2)}" ixy="0.0" ixz="0.0"
-                    iyy="${(1/12) * chassis_mass * (chassis_width**2 + chassis_height**2)}" iyz="0.0"
-                    izz="${(1/12) * chassis_mass * (chassis_width**2 + chassis_length**2)}"/>
+                    ixx="${(1/12) * chassis_mass * (3 * chassis_radius**2 + chassis_height**2)}" ixy="0.0" ixz="0.0"
+                    iyy="${(1/12) * chassis_mass * (3 * chassis_radius**2 + chassis_height**2)}" iyz="0.0"
+                    izz="${(1/2) * chassis_mass * (chassis_radius**2)}"/>
             </inertial>
             <visual>
                 <geometry>
-                    <box size="${chassis_width} ${chassis_length} ${chassis_height}"/>
+                    <cylinder radius="${chassis_radius}" length="${chassis_height}"/>
                 </geometry>
                 <origin xyz="0.0 0.0 0.0" rpy="0 0 0"/>
@@ -23,10 +22,7 @@
             <collision>
                 <geometry>
-                    <box size="${chassis_width} ${chassis_length} ${chassis_height}"/>
+                    <cylinder radius="${chassis_radius}" length="${chassis_height}"/>
                 </geometry>
                 <origin xyz="0.0 0.0 0.0" rpy="0 0 0"/>
-                <material name="white">
-                    <color rgba="1 1 1 1"/>
-                </material>
             </collision>
         </link>

File: sophia_description/urdf/mech/sophia_hexapod.urdf.xacro (robot description, xacro)
@@ -8,21 +8,25 @@
         <origin xyz="0 0 0.15" rpy="0 0 0"/> </joint>
     <xacro:prosoma_chassis base_link="base_link" prefix=""/>
+    <xacro:property name="rf_yaw" value="pi/3"/>
+    <xacro:macro name="origin_leg" params="yaw">
+        <origin xyz="${chassis_radius * cos(yaw)} ${chassis_radius * sin(yaw)} 0.0" rpy="0 0 ${yaw}"/>
+    </xacro:macro>
     <xacro:leg prefix="rf_" parent="base_link">
-        <origin xyz="0.06 0.08 0.0" rpy="0 0 ${pi/4}"/>
+        <xacro:origin_leg yaw="${pi/3}"/>
     </xacro:leg>
     <xacro:leg prefix="rm_" parent="base_link">
-        <origin xyz="0.06 0.0 0.0" rpy="0 0 0"/>
+        <xacro:origin_leg yaw="${0.0}"/>
     </xacro:leg>
     <xacro:leg prefix="rb_" parent="base_link">
-        <origin xyz="0.06 -0.08 0.0" rpy="0 0 ${-pi/4}"/>
+        <xacro:origin_leg yaw="${-pi/3}"/>
     </xacro:leg>
     <xacro:leg prefix="lf_" parent="base_link">
-        <origin xyz="-0.06 0.08 0.0" rpy="0 0 ${3*pi/4}"/>
+        <xacro:origin_leg yaw="${2*pi/3}"/>
     </xacro:leg>
     <xacro:leg prefix="lm_" parent="base_link">
-        <origin xyz="-0.06 0.0 0.0" rpy="0 0 ${pi}"/>
+        <xacro:origin_leg yaw="${pi}"/>
     </xacro:leg>
     <xacro:leg prefix="lb_" parent="base_link">
-        <origin xyz="-0.06 -0.08 0.0" rpy="0 0 ${5*pi/4}"/>
+        <xacro:origin_leg yaw="${4*pi/3}"/>
     </xacro:leg>
     <xacro:macro name="joint_gazebo" params="name">

Commit message: + effort

File: sophia_description/urdf/mech/leg.urdf.xacro (robot description, xacro)
@@ -1,6 +1,6 @@
 <?xml version="1.0"?>
 <robot xmlns:xacro="http://www.ros.org/wiki/xacro">
-    <xacro:property name="joint_effort" value="2.0"/>    <!-- N·m: ~5× max static gravitational torque per leg -->
-    <xacro:property name="joint_velocity" value="6.28"/>  <!-- rad/s: ~1 rev/s, realistic servo limit -->
+    <xacro:property name="joint_effort" value="5.0"/>    <!-- N·m: ~5× max static gravitational torque per leg -->
+    <xacro:property name="joint_velocity" value="12"/>  <!-- rad/s: ~1 rev/s, realistic servo limit -->
     <xacro:property name="joint_damping" value="0.3"/>    <!-- N·m·s/rad: smooth deceleration without oscillatory buildup -->
     <xacro:property name="joint_friction" value="0.1"/>   <!-- N·m: Coulomb friction prevents perturbation-driven creep -->
