Commit message: gazebo config params separated from xacro files

File: sophia_description/urdf/gazebo/gazebo_config.urdf.xacro (robot description, xacro)
@@ -1,9 +1,21 @@
 <?xml version="1.0"?>
 <robot xmlns:xacro="http://www.ros.org/wiki/xacro">
+    <xacro:macro name="leg_gazebo_config" params="prefix">
+        <gazebo reference="${prefix}tibia_link">
+          <mu1>1.5</mu1>
+          <mu2>1.5</mu2>
+          <kp>500000.0</kp>
+          <kd>10.0</kd>
+          <minDepth>0.002</minDepth>
+        </gazebo>
+        <xacro:material_visual ref_link="${prefix}coxa_link" ambient="1 1 1 1" diffuse="1 1 1 1" specular="1 1 1 1"/>
+        <xacro:material_visual ref_link="${prefix}femur_link" ambient="1 1 1 1" diffuse="1 1 1 1" specular="1 1 1 1"/>
+        <xacro:material_visual ref_link="${prefix}tibia_link" ambient="1 1 1 1" diffuse="1 1 1 1" specular="1 1 1 1"/>
+    </xacro:macro>
     <xacro:macro name="joint_gazebo" params="name">
         <joint name="${name}">
             <command_interface name="position">
-                <param name="min">-3.14</param>
-                <param name="max">3.14</param>
+                <param name="min">-1.57</param>
+                <param name="max">1.57</param>
             </command_interface>
             <state_interface name="position"/>
@@ -11,32 +23,34 @@
         </joint>
     </xacro:macro>
-    <xacro:macro name="gazebo_ros2_control_plugin">
-        <gazebo>
-            <plugin filename="gz_ros2_control-system" name="gz_ros2_control::GazeboSimROS2ControlPlugin">
-                <parameters>$(find sophia_controller)/config/sophia_controllers.yaml</parameters>
-                <ros>
-                    <remapping>/controller_manager/robot_description:=/robot_description</remapping>
-                </ros>
-            </plugin>
-        </gazebo>
-    </xacro:macro>
-    <xacro:macro name="leg_gazebo_material" params="link_name">
-        <gazebo reference="${link_name}">
-            <visual>
-                <material>
-                    <ambient>0.2 0.2 0.2 1.0</ambient>
-                    <diffuse>0.2 0.2 0.2 1.0</diffuse>
-                </material>
-            </visual>
-            <!-- Friction: high values needed for 0.69kg robot (low normal force per foot) -->
-            <mu1>5.0</mu1>
-            <mu2>5.0</mu2>
-        </gazebo>
-    </xacro:macro>
-    <xacro:macro name="leg_gazebo_config" params="prefix">
-        <xacro:leg_gazebo_material link_name="${prefix}coxa_link"/>
-        <xacro:leg_gazebo_material link_name="${prefix}femur_link"/>
-        <xacro:leg_gazebo_material link_name="${prefix}tibia_link"/>
-        <xacro:leg_gazebo_material link_name="${prefix}base_motor_link"/>
-    </xacro:macro>
+    <gazebo>
+        <plugin filename="gz_ros2_control-system" name="gz_ros2_control::GazeboSimROS2ControlPlugin">
+            <parameters>$(find sophia_controller)/config/sophia_controllers.yaml</parameters>
+            <ros>
+                <remapping>/controller_manager/robot_description:=/robot_description</remapping>
+            </ros>
+        </plugin>
+    </gazebo>
+    <ros2_control name="RobotSystem" type="system">
+        <hardware>
+            <plugin>gz_ros2_control/GazeboSimSystem</plugin>
+        </hardware>
+        <xacro:joint_gazebo name="rf_coxa_joint"/>
+        <xacro:joint_gazebo name="rf_coxa_link_to_rf_femur_link"/>
+        <xacro:joint_gazebo name="rf_femur_link_to_rf_tibia_link"/>
+        <xacro:joint_gazebo name="rm_coxa_joint"/>
+        <xacro:joint_gazebo name="rm_coxa_link_to_rm_femur_link"/>
+        <xacro:joint_gazebo name="rm_femur_link_to_rm_tibia_link"/>
+        <xacro:joint_gazebo name="rb_coxa_joint"/>
+        <xacro:joint_gazebo name="rb_coxa_link_to_rb_femur_link"/>
+        <xacro:joint_gazebo name="rb_femur_link_to_rb_tibia_link"/>
+        <xacro:joint_gazebo name="lf_coxa_joint"/>
+        <xacro:joint_gazebo name="lf_coxa_link_to_lf_femur_link"/>
+        <xacro:joint_gazebo name="lf_femur_link_to_lf_tibia_link"/>
+        <xacro:joint_gazebo name="lm_coxa_joint"/>
+        <xacro:joint_gazebo name="lm_coxa_link_to_lm_femur_link"/>
+        <xacro:joint_gazebo name="lm_femur_link_to_lm_tibia_link"/>
+        <xacro:joint_gazebo name="lb_coxa_joint"/>
+        <xacro:joint_gazebo name="lb_coxa_link_to_lb_femur_link"/>
+        <xacro:joint_gazebo name="lb_femur_link_to_lb_tibia_link"/>
+    </ros2_control>
 </robot>

File: sophia_description/urdf/mech/leg.urdf.xacro (robot description, xacro)
@@ -124,14 +124,4 @@
       <dynamics damping="${joint_damping}" friction="${joint_friction}"/>
     </joint>
-    <gazebo reference="${prefix}tibia_link">
-      <mu1>1.5</mu1>
-      <mu2>1.5</mu2>
-      <kp>500000.0</kp>
-      <kd>10.0</kd>
-      <minDepth>0.002</minDepth>
-    </gazebo>
-    <xacro:material_visual ref_link="${prefix}coxa_link" ambient="1 1 1 1" diffuse="1 1 1 1" specular="1 1 1 1"/>
-    <xacro:material_visual ref_link="${prefix}femur_link" ambient="1 1 1 1" diffuse="1 1 1 1" specular="1 1 1 1"/>
-    <xacro:material_visual ref_link="${prefix}tibia_link" ambient="1 1 1 1" diffuse="1 1 1 1" specular="1 1 1 1"/>
   </xacro:macro>
 </robot>

File: sophia_description/urdf/mech/sophia_hexapod.urdf.xacro (robot description, xacro)
@@ -1,6 +1,10 @@
 <?xml version="1.0"?>
 <robot name="sophia_hexapod" xmlns:xacro="http://wiki.ros.org/xacro">
+    <xacro:arg name="use_gazebo" default="false"/>
     <xacro:include filename="$(find sophia_description)/urdf/mech/prosoma_chassis.urdf.xacro" />
     <xacro:include filename="$(find sophia_description)/urdf/mech/leg.urdf.xacro" />
+    <xacro:if value="$(arg use_gazebo)">
+        <xacro:include filename="$(find sophia_description)/urdf/gazebo/gazebo_config.urdf.xacro" />
+    </xacro:if>
     <link name="base_footprint"/> <joint name="base_joint" type="fixed">
         <parent link="base_footprint"/>
@@ -30,44 +34,11 @@
         <xacro:origin_leg yaw="${4*pi/3}"/>
     </xacro:leg>
-    <xacro:macro name="joint_gazebo" params="name">
-        <joint name="${name}">
-            <command_interface name="position">
-                <param name="min">-1.57</param>
-                <param name="max">1.57</param>
-            </command_interface>
-            <state_interface name="position"/>
-            <state_interface name="velocity"/>
-        </joint>
-    </xacro:macro>
-    <gazebo>
-        <plugin filename="gz_ros2_control-system" name="gz_ros2_control::GazeboSimROS2ControlPlugin">
-            <parameters>$(find sophia_controller)/config/sophia_controllers.yaml</parameters>
-            <ros>
-                <remapping>/controller_manager/robot_description:=/robot_description</remapping>
-            </ros>
-        </plugin>
-    </gazebo>
-    <ros2_control name="RobotSystem" type="system">
-        <hardware>
-            <plugin>gz_ros2_control/GazeboSimSystem</plugin>
-        </hardware>
-        <xacro:joint_gazebo name="rf_coxa_joint"/>
-        <xacro:joint_gazebo name="rf_coxa_link_to_rf_femur_link"/>
-        <xacro:joint_gazebo name="rf_femur_link_to_rf_tibia_link"/>
-        <xacro:joint_gazebo name="rm_coxa_joint"/>
-        <xacro:joint_gazebo name="rm_coxa_link_to_rm_femur_link"/>
-        <xacro:joint_gazebo name="rm_femur_link_to_rm_tibia_link"/>
-        <xacro:joint_gazebo name="rb_coxa_joint"/>
-        <xacro:joint_gazebo name="rb_coxa_link_to_rb_femur_link"/>
-        <xacro:joint_gazebo name="rb_femur_link_to_rb_tibia_link"/>
-        <xacro:joint_gazebo name="lf_coxa_joint"/>
-        <xacro:joint_gazebo name="lf_coxa_link_to_lf_femur_link"/>
-        <xacro:joint_gazebo name="lf_femur_link_to_lf_tibia_link"/>
-        <xacro:joint_gazebo name="lm_coxa_joint"/>
-        <xacro:joint_gazebo name="lm_coxa_link_to_lm_femur_link"/>
-        <xacro:joint_gazebo name="lm_femur_link_to_lm_tibia_link"/>
-        <xacro:joint_gazebo name="lb_coxa_joint"/>
-        <xacro:joint_gazebo name="lb_coxa_link_to_lb_femur_link"/>
-        <xacro:joint_gazebo name="lb_femur_link_to_lb_tibia_link"/>
-    </ros2_control>
+    <xacro:if value="$(arg use_gazebo)">
+        <xacro:leg_gazebo_config prefix="rf_"/>
+        <xacro:leg_gazebo_config prefix="rm_"/>
+        <xacro:leg_gazebo_config prefix="rb_"/>
+        <xacro:leg_gazebo_config prefix="lf_"/>
+        <xacro:leg_gazebo_config prefix="lm_"/>
+        <xacro:leg_gazebo_config prefix="lb_"/>
+    </xacro:if>
 </robot>

Commit message: [FIXED] Twist error and smooth change of linear speed

File: sophia_description/urdf/gazebo/gazebo_config.urdf.xacro (robot description, xacro)
@@ -9,7 +9,7 @@
           <minDepth>0.002</minDepth>
         </gazebo>
-        <xacro:material_visual ref_link="${prefix}coxa_link" ambient="1 1 1 1" diffuse="1 1 1 1" specular="1 1 1 1"/>
-        <xacro:material_visual ref_link="${prefix}femur_link" ambient="1 1 1 1" diffuse="1 1 1 1" specular="1 1 1 1"/>
-        <xacro:material_visual ref_link="${prefix}tibia_link" ambient="1 1 1 1" diffuse="1 1 1 1" specular="1 1 1 1"/>
+        <xacro:material_visual ref_link="${prefix}coxa_link" ambient="0.05 0.05 0.05 1.0" diffuse="0.1 0.1 0.1 1.0" specular="0.1 0.1 0.1 1.0"/>
+        <xacro:material_visual ref_link="${prefix}femur_link" ambient="0.2 0.1 0.0 1.0" diffuse="1.0 0.4 0.0 1.0" specular="0.2 0.2 0.2 1.0"/>
+        <xacro:material_visual ref_link="${prefix}tibia_link" ambient="0.05 0.05 0.05 1.0" diffuse="0.1 0.1 0.1 1.0" specular="0.1 0.1 0.1 1.0"/>
     </xacro:macro>
     <xacro:macro name="joint_gazebo" params="name">
@@ -31,4 +31,5 @@
         </plugin>
     </gazebo>
+    <xacro:material_visual ref_link="base_link" ambient="0.05 0.05 0.05 1.0" diffuse="0.1 0.1 0.1 1.0" specular="0.1 0.1 0.1 1.0"/>
     <ros2_control name="RobotSystem" type="system">
         <hardware>

File: sophia_description/urdf/mech/leg.urdf.xacro (robot description, xacro)
@@ -38,4 +38,10 @@
     </gazebo>
   </xacro:macro>
+  <material name="black">
+    <color rgba="0.1 0.1 0.1 1.0"/>
+  </material>
+  <material name="orange">
+    <color rgba="1.0 0.5 0.0 1.0"/>
+  </material>
   <xacro:macro name="leg" params="prefix parent *origin">
     <link name="${prefix}coxa_link">
@@ -46,4 +52,5 @@
         </geometry>
         <origin xyz="${coxa_link_width/2} 0.0 0.0" rpy="0 0 0"/>
+        <material name="black"/>
       </visual>
       <collision>
@@ -61,4 +68,5 @@
         </geometry>
         <origin xyz="${femur_link_width/2} 0.0 0.0" rpy="0 0 0"/>
+        <material name="orange"/>
       </visual>
       <collision>
@@ -76,4 +84,5 @@
         </geometry>
         <origin xyz="${tibia_link_width/2} 0.0 0.0" rpy="0 0 0"/>
+        <material name="black"/>
       </visual>
       <collision name="${prefix}tibia_body_collision">

File: sophia_description/urdf/mech/prosoma_chassis.urdf.xacro (robot description, xacro)
@@ -19,4 +19,7 @@
                 </geometry>
                 <origin xyz="0.0 0.0 0.0" rpy="0 0 0"/>
+                <material name="black">
+                    <color rgba="0.1 0.1 0.1 1.0"/>
+                </material>
             </visual>
             <collision>

Commit message: Tuning gazebo parameters to avoid yaw drift

File: sophia_description/urdf/gazebo/gazebo_config.urdf.xacro (robot description, xacro)
@@ -3,9 +3,30 @@
     <xacro:macro name="leg_gazebo_config" params="prefix">
         <gazebo reference="${prefix}tibia_link">
-          <mu1>1.5</mu1>
-          <mu2>1.5</mu2>
-          <kp>500000.0</kp>
-          <kd>10.0</kd>
-          <minDepth>0.002</minDepth>
+          <!-- BULLET FEATHERSTONE reads friction ONLY from <bullet> tag.       -->
+          <!-- <mu1>/<mu2> top-level tags and <ode><mu> are silently IGNORED.   -->
+          <surface>
+            <bounce>
+              <restitution_coefficient>0.0</restitution_coefficient>
+              <threshold>0</threshold>
+            </bounce>
+            <friction>
+              <bullet>
+                <friction>0.5</friction>
+                <friction2>0.5</friction2>
+                <!-- rolling_friction MUST be 0 for sphere feet -->
+                <rolling_friction>0.0</rolling_friction>
+              </bullet>
+              <torsional>
+                <coefficient>0.0</coefficient>
+              </torsional>
+            </friction>
+            <contact>
+              <bullet>
+                <!-- split_impulse is CRITICAL to prevent violent yaw kicks -->
+                <split_impulse>true</split_impulse>
+                <split_impulse_penetration_threshold>-0.001</split_impulse_penetration_threshold>
+              </bullet>
+            </contact>
+          </surface>
         </gazebo>
         <xacro:material_visual ref_link="${prefix}coxa_link" ambient="0.05 0.05 0.05 1.0" diffuse="0.1 0.1 0.1 1.0" specular="0.1 0.1 0.1 1.0"/>
@@ -26,4 +47,7 @@
         <plugin filename="gz_ros2_control-system" name="gz_ros2_control::GazeboSimROS2ControlPlugin">
             <parameters>$(find sophia_controller)/config/sophia_controllers.yaml</parameters>
+            <!-- P-gain 0.7: time_constant=~14ms. Tighter tracking than 0.5
+                 without the bounce of 1.0. -->
+            <position_proportional_gain>0.7</position_proportional_gain>
             <ros>
                 <remapping>/controller_manager/robot_description:=/robot_description</remapping>

File: sophia_description/urdf/mech/leg.urdf.xacro (robot description, xacro)
@@ -1,8 +1,8 @@
 <?xml version="1.0"?>
 <robot xmlns:xacro="http://www.ros.org/wiki/xacro">
-    <xacro:property name="joint_effort" value="15.0"/>  <!-- max torque -->
-    <xacro:property name="joint_velocity" value="2.792527"/>
-    <xacro:property name="joint_damping" value="0.1"/>
-    <xacro:property name="joint_friction" value="0.01"/>
+    <xacro:property name="joint_effort" value="2.0"/>    <!-- N·m: ~5× max static gravitational torque per leg -->
+    <xacro:property name="joint_velocity" value="6.28"/>  <!-- rad/s: ~1 rev/s, realistic servo limit -->
+    <xacro:property name="joint_damping" value="0.3"/>    <!-- N·m·s/rad: smooth deceleration without oscillatory buildup -->
+    <xacro:property name="joint_friction" value="0.1"/>   <!-- N·m: Coulomb friction prevents perturbation-driven creep -->
     <xacro:property name="coxa_link_mass" value="0.05"/>
     <xacro:property name="coxa_link_width" value="0.035"/>
@@ -18,7 +18,7 @@
     <xacro:property name="tibia_link_depth" value="0.005"/>
     <xacro:property name="tibia_sphere_radius" value="${tibia_link_height/2}"/>
-    <xacro:macro name="link_inertial" params="m w h d">
+    <xacro:macro name="link_inertial" params="m w h d *origin">
         <inertial>
-            <origin xyz="0 0 0" rpy="0 0 0"/>
+            <xacro:insert_block name="origin"/>
             <mass value="${m}"/>
             <inertia ixx="${(m/12) * (h*h + d*d)}" ixy="0.0" ixz="0.0"
@@ -46,5 +46,7 @@
   <xacro:macro name="leg" params="prefix parent *origin">
     <link name="${prefix}coxa_link">
-      <xacro:link_inertial m="${coxa_link_mass}" w="${coxa_link_width}" h="${coxa_link_height}" d="${coxa_link_depth}"/>
+      <xacro:link_inertial m="${coxa_link_mass}" w="${coxa_link_width}" h="${coxa_link_height}" d="${coxa_link_depth}">
+        <origin xyz="${coxa_link_width/2} 0.0 0.0" rpy="0 0 0"/>
+      </xacro:link_inertial>
       <visual>
         <geometry>
@@ -62,5 +64,7 @@
     </link>
     <link name="${prefix}femur_link">
-      <xacro:link_inertial m="${femur_link_mass}" w="${femur_link_width}" h="${femur_link_height}" d="${femur_link_depth}"/>
+      <xacro:link_inertial m="${femur_link_mass}" w="${femur_link_width}" h="${femur_link_height}" d="${femur_link_depth}">
+        <origin xyz="${femur_link_width/2} 0.0 0.0" rpy="0 0 0"/>
+      </xacro:link_inertial>
       <visual>
         <geometry>
@@ -78,18 +82,23 @@
     </link>
     <link name="${prefix}tibia_link">
-      <xacro:link_inertial m="${tibia_link_mass}" w="${tibia_link_width}" h="${tibia_link_height}" d="${tibia_link_depth}"/>
+      <xacro:link_inertial m="${tibia_link_mass}" w="${tibia_link_width}" h="${tibia_link_height}" d="${tibia_link_depth}">
+        <origin xyz="${(tibia_link_width - tibia_sphere_radius)/2} 0.0 0.0" rpy="0 0 0"/>
+      </xacro:link_inertial>
       <visual>
-        <geometry>
-          <box size="${tibia_link_width} ${tibia_link_depth} ${tibia_link_height}"/>
-        </geometry>
-        <origin xyz="${tibia_link_width/2} 0.0 0.0" rpy="0 0 0"/>
-        <material name="black"/>
-      </visual>
-      <collision name="${prefix}tibia_body_collision">
         <geometry>
           <box size="${tibia_link_width - tibia_sphere_radius} ${tibia_link_depth} ${tibia_link_height}"/>
         </geometry>
         <origin xyz="${(tibia_link_width - tibia_sphere_radius)/2} 0.0 0.0" rpy="0 0 0"/>
-      </collision>
+        <material name="black"/>
+      </visual>
+      <visual>
+        <geometry>
+          <sphere radius="${tibia_sphere_radius}"/>
+        </geometry>
+        <origin xyz="${tibia_link_width - tibia_sphere_radius} 0.0 0.0" rpy="0 0 0"/>
+      </visual>
+      <!-- tibia_body_collision (box) REMOVED: caused spurious asymmetric contacts
+           inducing yaw torque. Only the sphere at the tip makes ground contact.  -->
+      <!-- SOLE contact point: sphere at the foot tip -->
       <collision name="${prefix}tibia_foot_collision">
         <geometry>
@@ -111,5 +120,5 @@
     <joint name="${prefix}coxa_joint" type="revolute">
       <axis xyz="0 0 1"/>
-      <limit effort="${joint_effort}" lower="-1.57" upper="1.57" velocity="${joint_velocity}"/>
+      <limit effort="${joint_effort}" lower="-1.0" upper="1.0" velocity="${joint_velocity}"/>
       <parent link="${prefix}base_motor_link"/>
       <child link="${prefix}coxa_link"/>
@@ -119,5 +128,7 @@
     <joint name="${prefix}coxa_link_to_${prefix}femur_link" type="revolute">
       <axis xyz="0 1 0"/>
-      <limit effort="${joint_effort}" lower="-2.5" upper="2.5" velocity="${joint_velocity}"/>
+      <!-- lower=-1.85: swing apex analysis shows -1.796 rad needed at max diagonal speed. -->
+      <!-- Was -1.77 rad (-101.4°); joint was hitting stop during diagonal walks.          -->
+      <limit effort="${joint_effort}" lower="-1.85" upper="1.57" velocity="${joint_velocity}"/>
       <parent link="${prefix}coxa_link"/>
       <child link="${prefix}femur_link"/>
@@ -127,5 +138,8 @@
     <joint name="${prefix}femur_link_to_${prefix}tibia_link" type="revolute">
       <axis xyz="0 1 0"/>
-      <limit effort="${joint_effort}" lower="-2.0" upper="2.0" velocity="${joint_velocity}"/>
+      <!-- upper=2.75 rad (157.6°): kinematic analysis shows max SWING APEX needs 2.667 rad. -->
+      <!-- Was 2.0 rad (114°): violated on EVERY step. Fixed to 2.5 still violated at apex. -->
+      <!-- 2.75 gives 5° margin above worst-case swing apex (2.667 rad for lm/lb legs).    -->
+      <limit effort="${joint_effort}" lower="-2.0" upper="2.75" velocity="${joint_velocity}"/>
       <parent link="${prefix}femur_link"/>
       <child link="${prefix}tibia_link"/>

Commit message: tuning gazebo parameters

File: sophia_description/urdf/gazebo/gazebo_config.urdf.xacro (robot description, xacro)
@@ -2,7 +2,7 @@
 <robot xmlns:xacro="http://www.ros.org/wiki/xacro">
     <xacro:macro name="leg_gazebo_config" params="prefix">
-        <gazebo reference="${prefix}tibia_link">
-          <!-- BULLET FEATHERSTONE reads friction ONLY from <bullet> tag.       -->
-          <!-- <mu1>/<mu2> top-level tags and <ode><mu> are silently IGNORED.   -->
+        <!-- Reference the named collision directly so URDF→SDF places <surface>
+             inside the correct <collision> element and not under <link>. -->
+        <gazebo reference="${prefix}tibia_foot_collision">
           <surface>
             <bounce>
@@ -12,7 +12,8 @@
             <friction>
               <bullet>
-                <friction>0.5</friction>
-                <friction2>0.5</friction2>
-                <!-- rolling_friction MUST be 0 for sphere feet -->
+                <!-- Bullet Featherstone reads friction ONLY from <bullet> tag.  -->
+                <!-- mu1/mu2 top-level and <ode><mu> are silently IGNORED.       -->
+                <friction>0.3</friction>
+                <friction2>0.3</friction2>
                 <rolling_friction>0.0</rolling_friction>
               </bullet>
@@ -47,7 +48,8 @@
         <plugin filename="gz_ros2_control-system" name="gz_ros2_control::GazeboSimROS2ControlPlugin">
             <parameters>$(find sophia_controller)/config/sophia_controllers.yaml</parameters>
-            <!-- P-gain 0.7: time_constant=~14ms. Tighter tracking than 0.5
-                 without the bounce of 1.0. -->
-            <position_proportional_gain>0.7</position_proportional_gain>
+            <!-- Internal P-gain: velocity = P × error × update_rate.
+                 At P=0.5, update_rate=100Hz: time_constant=20ms.
+                 1.0 was too aggressive and caused bouncing. 0.25 was too sluggish. -->
+            <position_proportional_gain>0.25</position_proportional_gain>
             <ros>
                 <remapping>/controller_manager/robot_description:=/robot_description</remapping>

Commit message: animation editor + greeting animation test

File: sophia_description/urdf/gazebo/gazebo_config.urdf.xacro (robot description, xacro)
@@ -14,6 +14,6 @@
                 <!-- Bullet Featherstone reads friction ONLY from <bullet> tag.  -->
                 <!-- mu1/mu2 top-level and <ode><mu> are silently IGNORED.       -->
-                <friction>0.3</friction>
-                <friction2>0.3</friction2>
+                <friction>0.5</friction>
+                <friction2>0.5</friction2>
                 <rolling_friction>0.0</rolling_friction>
               </bullet>

File: sophia_description/urdf/mech/leg.urdf.xacro (robot description, xacro)
@@ -101,5 +101,5 @@
            inducing yaw torque. Only the sphere at the tip makes ground contact.  -->
       <!-- SOLE contact point: sphere at the foot tip -->
-      <collision name="${prefix}tibia_foot_collision">
+      <collision>
         <geometry>
           <sphere radius="${tibia_sphere_radius}"/>
